File: sch/rev_2/divtiesus.kicad_sch (KiCad schematic)
At the start: 45 parts, among them J1 JTAG, J2 Joystick, J3 SD_Card, SW1 RESET, SW2 NMI, SW3 SW_DIP_x02, U1 EPM240T100, U2 628128, U3 28C64, U4 ESP-12E, U5 LM1117MP-3.3, U6 74HCT165D, X1 24MHz

Commit message: Cosmetic fix: change R1 footprint from C_0603 to R_0603 and update IBOM
Parts:
- R1: footprint Capacitor_SMD:C_0603_1608Metric -> Resistor_SMD:R_0603_1608Metric
- U2: value 628128 -> 628128
Changed lines of the file:
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@@
 			)
 		)
-		(property "Value" "628128 "
+		(property "Value" "628128"
 			(at 39.37 46.355 0)
 			(effects
@@
 			)
 		)
-		(property "Footprint" "Capacitor_SMD:C_0603_1608Metric"
+		(property "Footprint" "Resistor_SMD:R_0603_1608Metric"
 			(at 231.775 66.675 0)
 			(effects
